File: STM32-H757BIT6-Breakout.kicad_pcb (KiCad board)
At the start: 4 copper layers, 100 x 100 mm, 37 parts, among them J1 10129381-916001BLF, J10 10129381-916001BLF, J2 10129381-916001BLF, J3 10129381-916001BLF, J4 10129381-916001BLF, J5 10129381-916001BLF, J6 10129381-916001BLF, J7 10129381-916001BLF, J8 10129381-916001BLF, J9 10129381-916001BLF, U1 STM32H757BITx

Commit message: v1.1
Parts:
- removed J2, J5, J6, J7, J8: 10129381-916001BLF, 10129381-916001BLF:10129381-916001BLF
- added C27: 1uF, Capacitor_SMD:C_0603_1608Metric_Pad1.08x0.95mm_HandSolder, F.Cu at (122.6, 131.0)
- added C28: 47uF, Capacitor_SMD:C_0603_1608Metric_Pad1.08x0.95mm_HandSolder, F.Cu at (113.0, 133.4)
- added C29: 10uF, Capacitor_SMD:C_0603_1608Metric_Pad1.08x0.95mm_HandSolder, F.Cu at (106.5, 129.1)
- added C30: .1uF, Capacitor_SMD:C_0603_1608Metric_Pad1.08x0.95mm_HandSolder, F.Cu at (153.5, 64.5)
- added C31: .1uF, Capacitor_SMD:C_0603_1608Metric_Pad1.08x0.95mm_HandSolder, F.Cu at (134.6, 131.0)
- added C32: .1uF, Capacitor_SMD:C_0603_1608Metric_Pad1.08x0.95mm_HandSolder, F.Cu at (123.6, 137.2)
- added D2: 1N5819, Diode_THT:D_DO-41_SOD81_P10.16mm_Horizontal, F.Cu at (108.5, 132.4)
- added D3: LED, LED_SMD:LED_0603_1608Metric_Pad1.05x0.95mm_HandSolder, F.Cu at (134.5, 80.8)
- added D4: LED, LED_SMD:LED_0603_1608Metric_Pad1.05x0.95mm_HandSolder, F.Cu at (136.5, 80.8)
- added J11: 10129381-916001BLF, 10129381-916001BLF:10129381-916001BLF, F.Cu at (140.0, 70.0)
- added J12: 10129381-916001BLF, 10129381-916001BLF:10129381-916001BLF, F.Cu at (115.0, 87.5)
- added J13: 10129381-916001BLF, 10129381-916001BLF:10129381-916001BLF, F.Cu at (115.0, 112.5)
- added J14: 10129381-916001BLF, 10129381-916001BLF:10129381-916001BLF, F.Cu at (153.5, 135.0)
- added J15: 10129381-916001BLF, 10129381-916001BLF:10129381-916001BLF, F.Cu at (185.0, 120.0)
- added J16: 10129381-916001BLF, 10129381-916001BLF:10129381-916001BLF, F.Cu at (178.5, 140.0)
- added R1: 12.1k, Resistor_SMD:R_0603_1608Metric_Pad0.98x0.95mm_HandSolder, F.Cu at (126.6, 131.0)
- added R3: 50, Resistor_SMD:R_0603_1608Metric_Pad0.98x0.95mm_HandSolder, F.Cu at (131.0, 78.2)
- added R4: 50, Resistor_SMD:R_0603_1608Metric_Pad0.98x0.95mm_HandSolder, F.Cu at (131.0, 80.0)
- added R5: 900k, Resistor_SMD:R_0603_1608Metric_Pad0.98x0.95mm_HandSolder, F.Cu at (115.4, 139.5)
- added R6: 39k, Resistor_SMD:R_0603_1608Metric_Pad0.98x0.95mm_HandSolder, F.Cu at (120.5, 125.0)
- added R7: 100k, Resistor_SMD:R_0603_1608Metric_Pad0.98x0.95mm_HandSolder, F.Cu at (122.0, 125.0)
- added R8: 10k, Resistor_SMD:R_0603_1608Metric_Pad0.98x0.95mm_HandSolder, F.Cu at (124.1, 135.2)
- added U2: USB3300-EZK-TR, Snapeda:QFN32_5X5MC_MCH, F.Cu at (131.5, 135.5)
- added U3: TPS7A4700RGWT, Snapeda:RGW0020A-IPC_A, F.Cu at (117.0, 130.5)
- added U4: TUSB322I, Package_DFN_QFN:Texas_X2QFN-12_1.6x1.6mm_P0.4mm, F.Cu at (120.0, 138.8)
- added Y1: ECS-.327-CDX-1038, Snapeda:ECS-.327-CDX-1038_XTAL_ECS-.327-CDX-1038, F.Cu at (124.5, 92.5)
- added Y2: ECS-80-18-4X-CKM, Snapeda:ECS-80-18-4X-CKM_XTAL_ECS-80-18-4X-CKM, F.Cu at (124.0, 105.0)
- added Y3: ECS-240-20-4X, Snapeda:ECS-240-20-4X_XTAL_ECS-240-20-4X, F.Cu at (129.6, 126.5)
- J1: value 10129381-916001BLF -> GSB1C411111DS1HR; footprint 10129381-916001BLF:10129381-916001BLF -> Snapeda:GSB1C411111DS1HR_AMPHENOL_GSB1C411111DS1HR
- J3: value 10129381-916001BLF -> FTSH-107-01-F-DV-K-P-TR; footprint 10129381-916001BLF:10129381-916001BLF -> Snapeda:CONN_FTSH-107-01-F-DV-K-P-TR_SAI
- J4: value 10129381-916001BLF -> DM3AT-SF-PEJM5; footprint 10129381-916001BLF:10129381-916001BLF -> Snapeda:DM3AT-SF-PEJM5_HRS_DM3AT-SF-PEJM5; moved to B.Cu
- moved J4 85.6 mm to (191.4, 74.0), turned to -90 degrees
- moved J3 79.9 mm to (155.8, 58.0), turned to 180 degrees
- moved J1 71.8 mm to (120.2, 147.5), turned to 0 degrees
- moved J10 53.5 mm to (165.0, 70.0), turned to 180 degrees
- moved J9 13.2 mm to (185.0, 95.0), turned to -90 degrees
- moved C15 2.53 mm to (138.0, 117.5)
- moved C2 1.77 mm to (155.3, 118.4)
- moved C18 1.62 mm to (160.8, 117.4), turned to 90 degrees
- moved C8 1.12 mm to (168.0, 86.5)
- moved C5 1.12 mm to (168.4, 88.0)
- moved C7 1.04 mm to (140.0, 80.9)
- moved C3 1.00 mm to (168.4, 89.7)
- moved C1 0.95 mm to (141.6, 80.9)
- moved C26 0.86 mm to (134.5, 84.5)
- moved C13 0.60 mm to (132.4, 101.0)
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Connections:
- J10 pad 01: 3.3v -> Net-(U1-PH14)
- J10 pad 03: 3.3v -> Net-(U1-PI0)
- J10 pad 04: GND -> Net-(U1-PH15)
- J10 pad 05: 3.3v -> Net-(U1-PI2)
- J10 pad 06: GND -> Net-(U1-PI1)
- J10 pad 07: 3.3v -> Net-(U1-PD1)
- J10 pad 08: GND -> Net-(U1-PI3)
- J10 pad 09: 3.3v -> Net-(U1-PD3)
- J10 pad 10: GND -> Net-(U1-PD0)
- J10 pad 11: 3.3v -> Net-(U1-PD5)
- J10 pad 12: GND -> Net-(U1-PD4)
- J10 pad 13: 3.3v -> Net-(U1-PD7)
- J10 pad 14: GND -> Net-(U1-PD6)
- J10 pad 15: 3.3v -> Net-(U1-PG10)
- J10 pad 16: GND -> Net-(U1-PG9)
- J3 pad 10: Net-(U1-PB0) -> Net-(U1-PA15)
- J3 pad 11: Net-(U1-PA3) -> unconnected-(J3-Pad11)
- J3 pad 12: Net-(U1-PB1) -> Net-(U1-NRST)
- J3 pad 13: Net-(U1-PA4) -> Net-(U1-PB6)
- J3 pad 14: Net-(U1-PB2) -> Net-(U1-PB7)
- J9 pad 01: Net-(U1-PD11) -> Net-(U1-PH13)
- J9 pad 02: Net-(U1-PG5) -> GND
- J9 pad 03: Net-(U1-PD12) -> Net-(U1-PA12)
- J9 pad 04: Net-(U1-PG6) -> Net-(U1-PA11)
- J9 pad 05: Net-(U1-PD13) -> Net-(U1-PA10)
- J9 pad 06: Net-(U1-PG7) -> Net-(U1-PA9)
- J9 pad 07: Net-(U1-PD14) -> Net-(U1-PA8)
- J9 pad 08: Net-(U1-PG8) -> Net-(U1-PC7)
- J9 pad 09: Net-(U1-PD15) -> Net-(U1-PC6)
- J9 pad 10: Net-(U1-PC6) -> Net-(U1-PG8)
- J9 pad 11: Net-(U1-PG2) -> Net-(U1-PG7)
- J9 pad 12: Net-(U1-PC7) -> Net-(U1-PG6)
- J9 pad 13: Net-(U1-PG3) -> Net-(U1-PG5)
- J9 pad 14: Net-(U1-PC8) -> Net-(U1-PG4)
- J9 pad 15: Net-(U1-PG4) -> Net-(U1-PG3)
- J9 pad 16: Net-(U1-PC9) -> Net-(U1-PG2)
- U1 pad 144: Net-(U1-PC8) -> Net-(J4-DAT0)
- U1 pad 145: Net-(U1-PC9) -> Net-(J4-DAT1)
- U1 pad 167: Net-(U1-PC10) -> Net-(J4-DAT2)
- U1 pad 168: Net-(U1-PC11) -> Net-(J4-CD/DAT3)
- U1 pad 169: Net-(U1-PC12) -> Net-(J4-CLK)
- U1 pad 172: Net-(U1-PD2) -> Net-(J4-CMD)
Routing:
- net VBUS: track 0.00 -> 57.4 mm
- net Net-(U1-PB5): track 42.0 -> 96.8 mm, vias 1 -> 2
- net GND: track 101.5 -> 153.5 mm, vias 25 -> 47
- net Net-(J4-DAT1): track 0.00 -> 38.4 mm, vias 0 -> 1
- net Net-(U1-PC11): track 37.0 -> 0.00 mm
- net Net-(U1-PC12): track 36.7 -> 0.00 mm
- net Net-(J4-DAT0): track 0.00 -> 36.3 mm, vias 0 -> 1
- net Net-(J4-CLK): track 0.00 -> 36.2 mm, vias 0 -> 1
- net Net-(J4-CMD): track 0.00 -> 35.5 mm, vias 0 -> 1
- net Net-(U1-PC9): track 32.7 -> 0.00 mm
- net Net-(J4-CD/DAT3): track 0.00 -> 32.5 mm, vias 0 -> 1
- net Net-(U1-PA10): track 50.8 -> 19.1 mm
- net Net-(U1-PC8): track 31.2 -> 0.00 mm
- net Net-(J4-DAT2): track 0.00 -> 31.1 mm, vias 0 -> 1
- net Net-(U1-PD2): track 30.2 -> 0.00 mm, vias 1 -> 0
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Other:
- board text added: "H757 Breakout v1.1"
- board text removed: "3.3v"
- board text removed: "BOOT0"
- board text removed: "GND"
- board text removed: "NRST"
- board text removed: "PA0"
- board text removed: "PA1"
- board text removed: "PA10"
- board text removed: "PA11"
- board text removed: "PA12"
- board text removed: "PA13"
- board text removed: "PA14"
- board text removed: "PA15"
- board text removed: "PA8"
- board text removed: "PA9"
- board text removed: "PB10"
- board text removed: "PB11"
- board text removed: "PB12"
- board text removed: "PB13"
- board text removed: "PB14"
- board text removed: "PB15"
- board text removed: "PB3"
- board text removed: "PB4"
- board text removed: "PB5"
- board text removed: "PB6"
- board text removed: "PB7"
- board text removed: "PB8"
- board text removed: "PB9"
- board text removed: "PC0"
- board text removed: "PC1"
- board text removed: "PC10"
- board text removed: "PC11"
- board text removed: "PC12"
- board text removed: "PC13"
- board text removed: "PC14"
- board text removed: "PC15"
- board text removed: "PC2_C"
- board text removed: "PC3_C"
- board text removed: "PC6"
- board text removed: "PC7"
- board text removed: "PC8"
- board text removed: "PC9"
- board text removed: "PD0"
- board text removed: "PD1"
- board text removed: "PD10"
- board text removed: "PD11"
- board text removed: "PD12"
- board text removed: "PD13"
- board text removed: "PD14"
- board text removed: "PD15"
- board text removed: "PD2"
- board text removed: "PD3"
- board text removed: "PD4"
- board text removed: "PD5"
- board text removed: "PD6"
- board text removed: "PD7"
- board text removed: "PD8"
- board text removed: "PD9"
- board text removed: "PDR_ON"
- board text removed: "PE0"
- board text removed: "PE1"
- board text removed: "PE10"
- board text removed: "PE11"
- board text removed: "PE12"
- board text removed: "PE13"
- board text removed: "PE14"
- board text removed: "PE15"
- board text removed: "PE2"
- board text removed: "PE3"
- board text removed: "PE4"
- board text removed: "PE5"
- board text removed: "PE6"
- board text removed: "PE7"
- board text removed: "PE8"
- board text removed: "PE9"
- board text removed: "PF0"
- board text removed: "PF1"
- board text removed: "PF10"
- board text removed: "PF11"
- board text removed: "PF12"
- board text removed: "PF13"
- board text removed: "PF14"
- board text removed: "PF15"
- board text removed: "PF2"
- board text removed: "PF3"
- board text removed: "PF4"
- board text removed: "PF5"
- board text removed: "PF6"
- board text removed: "PF7"
- board text removed: "PF8"
- board text removed: "PF9"
- board text removed: "PG0"
- board text removed: "PG1"
- board text removed: "PG10"
- board text removed: "PG11"
- board text removed: "PG12"
- board text removed: "PG13"
- board text removed: "PG14"
- board text removed: "PG15"
- board text removed: "PG2"
- board text removed: "PG3"
- board text removed: "PG4"
- board text removed: "PG5"
- board text removed: "PG6"
- board text removed: "PG7"
- board text removed: "PG8"
- board text removed: "PG9"
- board text removed: "PH0"
- board text removed: "PH1"
- board text removed: "PH10"
- board text removed: "PH11"
- board text removed: "PH12"
- board text removed: "PH13"
- board text removed: "PH14"
- board text removed: "PH15"
- board text removed: "PH6"
- board text removed: "PH7"
- board text removed: "PH8"
- board text removed: "PH9"
- board text removed: "PI0"
- board text removed: "PI1"
- board text removed: "PI10"
- board text removed: "PI11"
- board text removed: "PI2"
- board text removed: "PI3"
- board text removed: "PI4"
- board text removed: "PI5"
- board text removed: "PI6"
- board text removed: "PI7"
- board text removed: "PI8"
- board text removed: "PI9"
