File: STM32-H757BIT6-Breakout.kicad_sch (KiCad schematic)
At the start: 37 parts, among them J1 10129381-916001BLF, J10 10129381-916001BLF, J2 10129381-916001BLF, J3 10129381-916001BLF, J4 10129381-916001BLF, J5 10129381-916001BLF, J6 10129381-916001BLF, J7 10129381-916001BLF, J8 10129381-916001BLF, J9 10129381-916001BLF, U1 STM32H757BITx

Commit message: v1.1
Parts:
- removed J1, J2, J3, J4, J5, J6, J7, J8: 10129381-916001BLF, 10129381-916001BLF:10129381-916001BLF, symbol 10129381-916001BLF:10129381-916001BLF
- added C27: 1uF, Capacitor_SMD:C_0603_1608Metric_Pad1.08x0.95mm_HandSolder, symbol Device:C_Small
- added C28: 47uF, Capacitor_SMD:C_0603_1608Metric_Pad1.08x0.95mm_HandSolder, symbol Device:C_Small
- added C29: 10uF, Capacitor_SMD:C_0603_1608Metric_Pad1.08x0.95mm_HandSolder, symbol Device:C_Small
- added C30, C31, C32: .1uF, Capacitor_SMD:C_0603_1608Metric_Pad1.08x0.95mm_HandSolder, symbol Device:C_Small
- added D2: 1N5819, Diode_THT:D_DO-41_SOD81_P10.16mm_Horizontal, symbol Diode:1N5819
- added D3, D4: LED, LED_SMD:LED_0603_1608Metric_Pad1.05x0.95mm_HandSolder, symbol Device:LED
- added J1: GSB1C411111DS1HR, Snapeda:GSB1C411111DS1HR_AMPHENOL_GSB1C411111DS1HR, symbol Snapeda:GSB1C411111DS1HR
- added J11, J12, J13, J14, J15, J16: 10129381-916001BLF, 10129381-916001BLF:10129381-916001BLF, symbol 10129381-916001BLF:10129381-916001BLF
- added J3: FTSH-107-01-F-DV-K-P-TR, Snapeda:CONN_FTSH-107-01-F-DV-K-P-TR_SAI, symbol Snapeda:FTSH-107-01-F-DV-K-P-TR
- added J4: DM3AT-SF-PEJM5, Snapeda:DM3AT-SF-PEJM5_HRS_DM3AT-SF-PEJM5, symbol Snapeda:DM3AT-SF-PEJM5
- added R1: 12.1k, Resistor_SMD:R_0603_1608Metric_Pad0.98x0.95mm_HandSolder, symbol Device:R_Small
- added R3, R4: 50, Resistor_SMD:R_0603_1608Metric_Pad0.98x0.95mm_HandSolder, symbol Device:R_Small
- added R5: 900k, Resistor_SMD:R_0603_1608Metric_Pad0.98x0.95mm_HandSolder, symbol Device:R_Small
- added R6: 39k, Resistor_SMD:R_0603_1608Metric_Pad0.98x0.95mm_HandSolder, symbol Device:R
- added R7: 100k, Resistor_SMD:R_0603_1608Metric_Pad0.98x0.95mm_HandSolder, symbol Device:R
- added R8: 10k, Resistor_SMD:R_0603_1608Metric_Pad0.98x0.95mm_HandSolder, symbol Device:R
- added U2: USB3300-EZK-TR, Snapeda:QFN32_5X5MC_MCH, symbol Snapeda:USB3300-EZK-TR
- added U3: TPS7A4700RGWT, Snapeda:RGW0020A-IPC_A, symbol Snapeda:TPS7A4700RGWT
- added U4: TUSB322I, Package_DFN_QFN:Texas_X2QFN-12_1.6x1.6mm_P0.4mm, symbol Interface_USB:TUSB322I
- added Y1: ECS-.327-CDX-1038, Snapeda:ECS-.327-CDX-1038_XTAL_ECS-.327-CDX-1038, symbol Snapeda:ECS-.327-CDX-1038
- added Y2: ECS-80-18-4X-CKM, Snapeda:ECS-80-18-4X-CKM_XTAL_ECS-80-18-4X-CKM, symbol Snapeda:ECS-80-18-4X-CKM
- added Y3: ECS-240-20-4X, Snapeda:ECS-240-20-4X_XTAL_ECS-240-20-4X, symbol Snapeda:ECS-240-20-4X
Connections:
- net 3.3v: now also C28.2, C31.1, J16.01, J16.02, J16.03, J16.04, J16.05, J16.06, J16.07, J16.08, J16.09, J16.10, J16.12, J16.14, J16.16, J3.3, J4.4 (VDD), R3.2, R4.2, U2.25 (VDD3.3), U2.30 (VDD3.3), U2.31 (REG_EN), U3.1 (OUT), U3.20 (OUT), U3.3 (SENSE_FB), U4.12 (VDD); no longer J10.01, J10.03, J10.05, J10.07, J10.09, J10.11, J10.13, J10.15
- net GND: now also J9.02, C27.1, C28.1, C29.1, C30.2, C31.2, C32.2, J1.A1B12 (GND_A), J1.B1A12 (GND_B), J1.SH1 (SHIELD), J1.SH2 (SHIELD__1), J1.SH3 (SHIELD__2), J1.SH4 (SHIELD__3), J11.01, J11.02, J12.02, J13.02, J14.02, J15.02, J3.5, J3.7, J4.6 (VSS), J4.P1 (SHIELD), J4.P2 (SHIELD__1), J4.P3 (SHIELD__2), J4.P4 (SHIELD__3), R1.2, R6.1, U2.1 (GND), U2.2 (GND), U2.3 (CPEN), U2.33 (EPAD), U3.12 (0P1V), U3.21 (Thermal_Pad), U3.6 (3P2V), U3.7 (GND), U4.10 (GND), U4.5 (ADDR); no longer J10.04, J10.06, J10.08, J10.10, J10.12, J10.14, J10.16
- net at U1.146 (PA8): now also J9.07
- net at U1.158 (PH15): now also J10.04
- net at U1.147 (PA9): now also J9.06
- net at U1.159 (PI0): now also J10.03
- net at U1.148 (PA10): now also J9.05
- net at U1.162 (PI1): now also J10.06
- net at U1.149 (PA11): now also J9.04
- net at U1.163 (PI2): now also J10.05
- net at U1.150 (PA12): now also J9.03
- net at U1.164 (PI3): now also J10.08
- net at U1.151 (PA13): now also J3.4
- net at U1.165 (PA14): now also J3.6
- net at U1.156 (PH13): now also J9.01
- net at U1.166 (PA15): now also J3.10
- net at U1.157 (PH14): now also J10.01
- net at U1.167 (PC10): now also J4.1 (DAT2)
- net at U1.26 (PF4): now also J12.15
- net at U1.36 (PH1): now also Y2.1
- net at U1.27 (PF5): now also J13.01
- net at U1.37 (NRST): now also C30.1, J3.12
- net at U1.30 (PF6): now also J13.04
- net at U1.38 (PC0): now also U2.13 (STP)
- net at U1.31 (PF7): now also J13.03
- net at U1.39 (PC1): now also J13.08
- net at U1.32 (PF8): now also J13.05
- net at U1.40 (PC2_C): now also U2.12 (DIR)
- net at U1.33 (PF9): now also J13.06
- net at U1.41 (PC3_C): now also U2.11 (NXT)
- net at U1.34 (PF10): now also J13.07
- net at U1.45 (PA0): now also J13.09
- net at U1.35 (PH0): now also Y2.2
- net at U1.46 (PA1): now also J13.10
- net at U1.188 (PG15): now also J11.08
- net at U1.196 (PB9): now also J11.12
- net at U1.189 (PB3): now also J3.8
- net at U1.197 (PE0): now also J11.11
- net at U1.190 (PB4): now also J11.07
- net at U1.198 (PE1): now also J11.14
- net at U1.191 (PB5): now also U2.17 (DATA7)
- net at U1.201 (PDR_ON): now also J11.13
- net at U1.192 (PB6): now also J3.13
- net at U1.203 (PI4): now also J11.16
- net at U1.193 (PB7): now also J3.14
- net at U1.204 (PI5): now also J11.15
- net at U1.194 (BOOT0): now also J11.10
- net at U1.205 (PI6): now also D4.1 (K)
- net at U1.195 (PB8): now also J11.09
- net at U1.206 (PI7): now also D3.1 (K)
- net at U1.47 (PA2): now also J13.11
- net at U1.59 (PA6): now also J14.15
- net at U1.48 (PH2): now also J13.12
- net at U1.60 (PA7): now also J14.16
- net at U1.51 (PH3): now also J13.13
- net at U1.61 (PC4): now also J14.13
- net at U1.52 (PH4): now also J13.14
- net at U1.62 (PC5): now also J14.14
- net at U1.53 (PH5): now also J13.16
- net at U1.63 (PB0): now also U2.23 (DATA1)
- net at U1.54 (PA3): now also U2.24 (DATA0)
- net at U1.64 (PB1): now also U2.22 (DATA2)
- net at U1.57 (PA4): now also J13.15
- net at U1.65 (PB2): now also J14.11
- net at U1.58 (PA5): now also U2.14 (CLKOUT)
- net at U1.66 (PI15): now also J14.12
- net at U1.1 (PE2): now also J12.01
- net at U1.12 (PC15): now also Y1.2
- net at U1.2 (PE3): now also J12.04
- net at U1.13 (PI9): now also J12.10
- net at U1.3 (PE4): now also J12.03
- net at U1.14 (PI10): now also J12.09
- net at U1.4 (PE5): now also J12.06
- net at U1.15 (PI11): now also J12.12
- net at U1.5 (PE6): now also J12.05
- net at U1.22 (PF0): now also J12.11
- net at U1.9 (PI8): now also J12.08
- net at U1.23 (PF1): now also J12.14
- net at U1.10 (PC13): now also J12.07
- net at U1.24 (PF2): now also J12.13
- net at U1.11 (PC14): now also Y1.1
- net at U1.25 (PF3): now also J12.16
- net at U1.87 (PB10): now also U2.21 (DATA3)
- net at U1.98 (PH12): now also J15.12
- net at U1.88 (PB11): now also U2.20 (DATA4)
- net at U1.101 (PB12): now also U2.19 (DATA5)
- net at U1.92 (PH6): now also J16.11
- net at U1.102 (PB13): now also U2.18 (DATA6)
- net at U1.93 (PH7): now also J16.13
- net at U1.103 (PB14): now also J15.11
- net at U1.94 (PH8): now also J15.16
- net at U1.104 (PB15): now also J15.10
- net at U1.95 (PH9): now also J15.15
- net at U1.105 (PD8): now also J15.09
- net at U1.96 (PH10): now also J15.14
- net at U1.106 (PD9): now also J15.08
- net at U1.97 (PH11): now also J15.13
- net at U1.107 (PD10): now also J15.07
- net at U1.67 (PF11): now also J14.09
- net at U1.77 (PE8): now also J14.07
- net at U1.68 (PF12): now also U4.11 (~{EN})
- net at U1.78 (PE9): now also J14.08
- net at U1.69 (PF13): now also U2.9 (RESET)
- net at U1.81 (PE10): now also J14.05
- net at U1.70 (PF14): now also U4.8 (SCL/OUT2)
- net at U1.82 (PE11): now also J14.06
- net at U1.71 (PF15): now also U4.7 (SDA/OUT1)
- net at U1.83 (PE12): now also J14.03
- net at U1.72 (PG0): now also R6.2, R7.1
- net at U1.84 (PE13): now also J14.04
- net at U1.75 (PG1): now also U4.6 (~{INT}/OUT3)
- net at U1.85 (PE14): now also J14.01
- net at U1.76 (PE7): now also J14.10
- net at U1.86 (PE15): now also J16.15
- net at U1.168 (PC11): now also J4.2 (CD/DAT3)
- net at U1.176 (PD6): now also J10.14
- net at U1.169 (PC12): now also J4.5 (CLK)
- net at U1.177 (PD7): now also J10.13
- net at U1.170 (PD0): now also J10.10
- net at U1.180 (PG9): now also J10.16
- net at U1.171 (PD1): now also J10.07
- net at U1.181 (PG10): now also J10.15
- net at U1.172 (PD2): now also J4.3 (CMD)
- net at U1.182 (PG11): now also J11.04
- net at U1.173 (PD3): now also J10.09
- net at U1.183 (PG12): now also J11.03
- net at U1.174 (PD4): now also J10.12
- net at U1.184 (PG13): now also J11.06
- net at U1.175 (PD5): now also J10.11
- net at U1.185 (PG14): now also J11.05
- net at U1.110 (PD11): now also J15.06; no longer J9.01
- net at U1.135 (PG5): now also J9.13; no longer J9.02
- net at U1.111 (PD12): now also J15.05; no longer J9.03
- net at U1.136 (PG6): now also J9.12; no longer J9.04
- net at U1.112 (PD13): now also J15.04; no longer J9.05
- net at U1.137 (PG7): now also J9.11; no longer J9.06
- net at U1.115 (PD14): now also J15.03; no longer J9.07
- net at J9.08: now also U1.143 (PC7); no longer U1.138 (PG8)
- net at J9.09: now also U1.142 (PC6); no longer U1.116 (PD15)
- net at J9.10: now also U1.138 (PG8); no longer U1.142 (PC6)
- net at U1.130 (PG2): now also J9.16; no longer J9.11
- net at U1.131 (PG3): now also J9.15; no longer J9.13
- net at U1.144 (PC8): now also J4.7 (DAT0); no longer J9.14
- net at U1.134 (PG4): now also J9.14; no longer J9.15
- net at U1.145 (PC9): now also J4.8 (DAT1); no longer J9.16
- new net: U2.27 (XO), Y3.1
- new net: U2.28 (XI), Y3.2
- new net: D3.2 (A), R4.1
- new net: D4.2 (A), R3.1
- new net: C32.1, U2.16 (VDD3.3), U2.6 (VDD3.3)
- new net: R1.1, U2.32 (RBIAS)
- new net: R8.1, U2.4 (VBUS)
- new net: U2.5 (ID), U4.9 (ID)
- new net: R5.2, U4.3 (VBUS_DET)
- new net: J1.A5 (CC1), U4.1 (CC1)
- new net: J1.B5 (CC2), U4.2 (CC2)
- new net: C29.2, D2.1 (K), U3.13 (EN), U3.15 (IN), U3.16 (IN)
- new net: C27.2, U3.14 (NR)
- new net: J15.01, U1.116 (PD15)
- new net USB_DN: J1.A7 (D1-), U2.8 (DM)
- new net USB_DP: J1.A6 (D1+), U2.7 (DP)
- new net VBUS: D2.2 (A), J1.A4B9 (VBUS_A), J1.B4A9 (VBUS_B), R5.1, R7.2, R8.2
- no-connect marks 16 -> 41
Other:
- moved on the sheet: C1, C10, C11, C12, C13, C14, C15, C16, C17, C18, C19, C2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
